File: PCB_Controller/PCB_Controller.kicad_pcb (KiCad board)
At the start: 2 copper layers, 304.1 x 203.1 mm, 141 parts, among them J1 ATX_Pin_fromPSU, J10 Conn_01x15, J11 Conn_01x15, J2 ColumnPin_1-12, J3 ColumnPin_13-24, J4 ColumnPin_25-36, J5 RowPin_1-8, J6 RowPin_9-16, J7 RowPin17-24, J8 Conn_01x05, Q2 ULN2803APG_O,N,HZN, Q3 ULN2803APG_O,N,HZN, Q4 ULN2803APG_O,N,HZN, Q5 ULN2803APG_O,N,HZN, Q6 ULN2803APG_O,N,HZN, Q7 ULN2803APG_O,N,HZN, Q8 ULN2803APG_O,N,HZN, Q9 ULN2803APG_O,N,HZN, U10 74HC595, U11 74HC595, U12 74HC595, U13 74HC595, U14 74HC595, U15 UDN2981A, U16 UDN2981A, U17 UDN2981A, U18 UDN2981A, U19 UDN2981A, U20 SN74HC75N, U22 74HC00, U23 ESP32-DEVKIT-V1, U25 74HC595, U26 74HC595, U27 74HC595, U30 74HC595, U31 74HC595, U32 74HC595, U33 UDN2981A, U34 UDN2981A, U35 UDN2981A, U5 74HC595, U6 74HC595, U7 74HC595, U8 74HC595, U9 74HC595

Commit message: Power the controller from a 24 V jack and shrink the board to 249x122 mm
- The ATX 20-pin input is gone. A 24 V barrel jack (CUI PJ-063AH, 8 A)
  feeds the coil drivers directly, with a 470 uF bulk cap. A TRACO
  TSR 1-2450 makes 5 V for the ESP32's VIN; the DevKit's 3V3 pin feeds
  the +3.3V logic rail. VIN used to sit on 3.3 V, which starved the
  DevKit's own regulator.
- One ground: GND2 was the ATX -12 V rail, which left the ULN2803
  emitters 12 V below the 74HC595 outputs driving them.
- The coil rail is +24V (was +12V). The PSU-status LED now shows 5 V,
  through 2.2k.
- PULSE moves to GPIO32 and SET/RST to GPIO33: GPIO34/35 are input-only
  and could not drive U22/U20.
- New layout, 249x122 mm (was 304x203): 16 channel strips of driver,
  pull-downs and 74HC595, the six IDC headers along the top edge, the
  ESP32 and power entry on the left. Autorouted with Freerouting, GND
  poured on both layers. Net classes: +24V 1.0 mm, GND 0.8 mm, coil
  lines 0.6 mm, logic power 0.5 mm, signals 0.3 mm, 0.3 mm clearance.
- DRC: no errors, nothing unconnected, matches the schematic.

Co-Authored-By: Claude Opus 5.5 <noreply@anthropic.com>
Parts:
- added C1: 470uF/35V, Capacitor_THT:CP_Radial_D10.0mm_P5.00mm, F.Cu at (119.0, 136.5)
- added C3: 10uF/50V, Capacitor_SMD:C_1206_3216Metric_Pad1.33x1.80mm_HandSolder, F.Cu at (113.5, 150.5)
- added C4: 22uF/10V, Capacitor_SMD:C_1206_3216Metric_Pad1.33x1.80mm_HandSolder, F.Cu at (132.5, 150.5)
- added U1: TSR_1-2450, Converter_DCDC:Converter_DCDC_TRACO_TSR-1_THT, F.Cu at (121.5, 152.3)
- D1: value LED_PSU_Status -> LED_Power_5V
- J1: value ATX_Pin_fromPSU -> 24V_DC_Jack; footprint ATX:39-29-920Y -> Connector_BarrelJack:BarrelJack_CUI_PJ-063AH_Horizontal
- R1: value 10k -> 2.2k
- moved Q7 165.8 mm to (279.0, 92.2), turned to 0 degrees
- moved Q8 159.6 mm to (301.8, 92.2), turned to 0 degrees
- moved C35 157.9 mm to (280.0, 160.5), turned to 0 degrees
- moved C16 154.8 mm to (165.7, 160.5), turned to 0 degrees
- moved Q9 154.1 mm to (324.7, 92.2), turned to 0 degrees
- moved C15 152.2 mm to (188.6, 160.5), turned to 0 degrees
- moved C36 150.7 mm to (302.9, 160.5), turned to 0 degrees
- moved C14 149.7 mm to (211.4, 160.5), turned to 0 degrees
- moved U32 148.6 mm to (279.3, 147.4), turned to 0 degrees
- moved C38 148.3 mm to (280.0, 106.2), turned to 0 degrees
- moved C37 144.6 mm to (325.7, 160.5), turned to 0 degrees
- moved C39 141.9 mm to (302.9, 106.2), turned to 0 degrees
- moved U31 141.7 mm to (302.1, 147.4), turned to 0 degrees
- moved J2 138.1 mm to (167.0, 62.8)
- moved C40 136.2 mm to (325.7, 106.2), turned to 0 degrees
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Connections:
- C17 pad 1: GND2 -> GND1
- C17 pad 2: +12V -> +24V
- C18 pad 1: GND2 -> GND1
- C18 pad 2: +12V -> +24V
- C19 pad 1: GND2 -> GND1
- C19 pad 2: +12V -> +24V
- C20 pad 1: GND2 -> GND1
- C20 pad 2: +12V -> +24V
- C21 pad 1: +12V -> +24V
- C21 pad 2: GND2 -> GND1
- C22 pad 1: GND2 -> GND1
- C22 pad 2: +12V -> +24V
- C23 pad 1: GND2 -> GND1
- C23 pad 2: +12V -> +24V
- C24 pad 1: GND2 -> GND1
- C24 pad 2: +12V -> +24V
- C25 pad 1: GND2 -> GND1
- C25 pad 2: +12V -> +24V
- C26 pad 1: +12V -> +24V
- C26 pad 2: GND2 -> GND1
- C29 pad 1: +12V -> +24V
- C29 pad 2: GND2 -> GND1
- C30 pad 1: +12V -> +24V
- C30 pad 2: GND2 -> GND1
- C31 pad 1: +12V -> +24V
- C31 pad 2: GND2 -> GND1
- C38 pad 1: +12V -> +24V
- C38 pad 2: GND2 -> GND1
- C39 pad 1: +12V -> +24V
- C39 pad 2: GND2 -> GND1
- C40 pad 1: GND2 -> GND1
- C40 pad 2: +12V -> +24V
- J1 pad 1: +3.3V -> +24V
- J1 pad 2: +3.3V -> GND1
- J10 pad 10: /D32 -> /Pulse
- J10 pad 11: /Set_Reset -> /D35
- J10 pad 12: /Pulse -> /D34
- J10 pad 9: /D33 -> /Set_Reset
- J11 pad 1: Net-(J11-Pin_1) -> +3.3V
- J8 pad 3: +12V -> +24V
- J8 pad 5: GND2 -> GND1
- Q2 pad 10: +12V -> +24V
- Q2 pad 9: GND2 -> GND1
- Q3 pad 10: +12V -> +24V
- Q3 pad 9: GND2 -> GND1
- Q4 pad 10: +12V -> +24V
- Q4 pad 9: GND2 -> GND1
- Q5 pad 10: +12V -> +24V
- Q5 pad 9: GND2 -> GND1
- Q6 pad 10: +12V -> +24V
- Q6 pad 9: GND2 -> GND1
- Q7 pad 10: +12V -> +24V
- Q7 pad 9: GND2 -> GND1
- Q8 pad 10: +12V -> +24V
- Q8 pad 9: GND2 -> GND1
- Q9 pad 10: +12V -> +24V
- Q9 pad 9: GND2 -> GND1
- R1 pad 1: /Checker -> +5V
- U15 pad 10: GND2 -> GND1
- U15 pad 9: +12V -> +24V
- U16 pad 10: GND2 -> GND1
- U16 pad 9: +12V -> +24V
- U17 pad 10: GND2 -> GND1
- U17 pad 9: +12V -> +24V
- U18 pad 10: GND2 -> GND1
- U18 pad 9: +12V -> +24V
- U19 pad 10: GND2 -> GND1
- U19 pad 9: +12V -> +24V
- U23 pad 1: Net-(J11-Pin_1) -> +3.3V
- U23 pad 19: /Pulse -> /D34
- U23 pad 20: /Set_Reset -> /D35
- U23 pad 21: /D32 -> /Pulse
- U23 pad 22: /D33 -> /Set_Reset
- U23 pad 30: +3.3V -> +5V
- U33 pad 10: GND2 -> GND1
- U33 pad 9: +12V -> +24V
- U34 pad 10: GND2 -> GND1
- U34 pad 9: +12V -> +24V
- U35 pad 10: GND2 -> GND1
- U35 pad 9: +12V -> +24V
Routing:
- net GND2: track 950.3 -> 0.00 mm, vias 9 -> 0
- net +3.3V: track 1474.1 -> 597.2 mm, vias 19 -> 1
- net +12V: track 869.3 -> 0.00 mm, vias 5 -> 0
- net /Clock: track 858.1 -> 271.3 mm, vias 5 -> 0
- net GND1: track 1584.7 -> 1014.9 mm
- net /Clear: track 781.7 -> 330.6 mm, vias 9 -> 2
- net +24V: track 0.00 -> 337.4 mm
- net Net-(U30-~{OE}): track 567.2 -> 244.6 mm, vias 7 -> 1
- net /Data: track 405.0 -> 191.3 mm, vias 6 -> 1
- net Net-(U10-~{OE}): track 364.1 -> 175.0 mm
- net Net-(U25-~{OE}): track 380.2 -> 217.3 mm, vias 1 -> 0
- net /Column_Latch: track 371.1 -> 218.5 mm, vias 6 -> 4
- net Net-(U11-SER): track 178.7 -> 31.0 mm, vias 0 -> 1
- net Col1: track 149.6 -> 33.2 mm
- net Col9: track 153.8 -> 52.6 mm
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Other:
- board size 304.1 x 203.1 mm -> 249.4 x 122 mm
- board text added: "(+) center"
- board text added: "+24V"
- board text added: "24V DC IN"
- board text added: "24V FLIP-DISC - NOT HUB75 LED"
- board text added: "D34"
- board text added: "D35"
- board text added: "ESP32 DevKit V1"
- board text removed: "+12V"
- board text removed: "10k Pull-down Resistor"
- board text removed: "12V FLIP-DISC - NOT HUB75 LED"
- board text removed: "3V3"
- board text removed: "74hc595"
- board text removed: "Column SINK drivers (1)"
- board text removed: "Column SOURCE drivers (1)"
- board text removed: "Column SOURCE drivers (2)"
- board text removed: "D32"
- board text removed: "D33"
- board text removed: "ESP32 Devkit"
- board text removed: "GND2(-12V)"
- board text removed: "Row SINK drivers"
- board text removed: "Row SOURCE drivers"
- board text removed: "Signal out"

Commit message: Add a 3.3 V LDO and a 24 V screw terminal to the controller power input
- J1 is now a 5.5 x 2.5 mm jack (CUI PJ-063BH, 8 A) to match 24 V
  10 A / 20 A adapter plugs; same land pattern as before
- J9: 2-pole 5.08 mm screw terminal in parallel with J1 for supplies
  with bare leads
- U2 AMS1117-3.3 (C5/C7) makes the +3.3V logic rail from +5V for the
  74HC595s, 74HC00 and 74HC75, instead of borrowing the DevKit's LDO
- The DevKit 3V3 pin is off the board rail (broken out on J11.1 only)
- J10.1, which sits on the ESP32 VIN pin, is now on +5V like VIN
- Re-placed and re-routed with Freerouting: DRC 0 errors, 0 unconnected

Co-Authored-By: Claude Opus 5.5 <noreply@anthropic.com>
Parts:
- added C5: 10uF/16V, Capacitor_SMD:C_1206_3216Metric_Pad1.33x1.80mm_HandSolder, F.Cu at (134.5, 162.5)
- added C7: 22uF/10V, Capacitor_SMD:C_1206_3216Metric_Pad1.33x1.80mm_HandSolder, F.Cu at (148.5, 162.5)
- added J9: Screw_Terminal_24V, TerminalBlock_Phoenix:TerminalBlock_Phoenix_MKDS-1,5-2-5.08_1x02_P5.08mm_Horizontal, F.Cu at (105.7, 150.0)
- added U2: AMS1117-3.3, Package_TO_SOT_SMD:SOT-223-3_TabPin2, F.Cu at (141.5, 162.5)
- J1: value 24V_DC_Jack -> DC_Jack_5.5x2.5_24V
Connections:
- J10 pad 1: +3.3V -> +5V
- J11 pad 1: +3.3V -> Net-(J11-Pin_1)
- U23 pad 1: +3.3V -> Net-(J11-Pin_1)
Routing:
- net +3.3V: track 597.2 -> 524.8 mm, vias 1 -> 3
- net +5V: track 109.6 -> 150.1 mm, vias 0 -> 1
- net Net-(U18-IN8): track 102.7 -> 67.5 mm, vias 6 -> 0
- net Col31: track 59.1 -> 92.9 mm, vias 1 -> 2
- net Net-(Q4-I6): track 92.4 -> 61.2 mm, vias 6 -> 1
- net GND1: track 1014.9 -> 1045.0 mm, vias 7 -> 5
- net /Clear: track 330.6 -> 301.4 mm, vias 2 -> 3
- net /Clock: track 271.3 -> 298.6 mm
- net Net-(U30-~{OE}): track 244.6 -> 217.7 mm
- net Net-(Q9-I7): track 55.8 -> 82.2 mm
- net Net-(U25-QA): track 63.9 -> 90.1 mm, vias 0 -> 2
- net Net-(U15-IN3): track 84.2 -> 61.4 mm
- net +24V: track 337.4 -> 359.5 mm, vias 0 -> 1
- net Net-(U26-QA): track 88.1 -> 66.1 mm, vias 3 -> 1
- net Col20: track 85.7 -> 64.5 mm, vias 3 -> 1
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Other:
- board text added: "1:+24V 2:GND"
- board text added: "24V IN"
- board text added: "24V IN 5.5x2.5"
- board text added: "3.3V LDO"
- board text added: "3V3"
- board text removed: "24V DC IN"

Commit message: Buffer the ESP32, cap coil pulses in hardware and protect the 24 V input
- U4 74HCT245 turns the ESP32's 3.3 V control lines into 5 V for all
  logic, so the 595s, 74HC00 and 74HC123 can be HC or HCT parts
- All logic now runs on +5V (74HC595 at 3.3 V could not drive a ULN2803
  channel to the ~0.5 A a coil pulse needs); AMS1117 and the 3.3 V rail
  are gone, J8 pin 1 / J11 pin 1 break out the DevKit's own 3V3
- U3 74HC123 one-shot: drivers see PULSE for at most ~2 ms (R40/C8)
- 10k pull-downs on PULSE and SET/RST keep the drivers off at boot
- 74HC75 (latch tied transparent) replaced by a spare 74HC00 gate
- Input: PPTC 3 A (F1), SMBJ28CA TVS (D2), IRF4905 reverse-polarity
  switch (Q1, D3 15 V zener, R41), 1000 uF bulk (C42)
- All 35 ICs on standard DIP socket footprints (the old 595 footprint
  had 7.94 mm rows), socket pads 1.4 mm to leave routing room
- Keepouts around the mounting holes; re-placed and re-routed, board
  kept at the position it was moved to in KiCad
- DRC 0 errors / 0 unconnected / 0 parity, ERC 0 errors
- ref/: the single-dot current pulse the limiter is sized for

Co-Authored-By: Claude Opus 5.5 <noreply@anthropic.com>
Parts:
- removed C5: 10uF/16V, Capacitor_SMD:C_1206_3216Metric_Pad1.33x1.80mm_HandSolder
- removed C7: 22uF/10V, Capacitor_SMD:C_1206_3216Metric_Pad1.33x1.80mm_HandSolder
- removed U2: AMS1117-3.3, Package_TO_SOT_SMD:SOT-223-3_TabPin2
- removed U20: SN74HC75N, SN74HC75N:7475
- added C41: 100nF, Capacitor_SMD:C_0805_2012Metric_Pad1.18x1.45mm_HandSolder, F.Cu at (79.9, 114.7)
- added C42: 1000uF/35V, Capacitor_THT:CP_Radial_D12.5mm_P5.00mm, F.Cu at (73.4, 47.7)
- added C43: 100nF, Capacitor_SMD:C_0805_2012Metric_Pad1.18x1.45mm_HandSolder, F.Cu at (62.9, 46.7)
- added C8: 100nF, Capacitor_SMD:C_0805_2012Metric_Pad1.18x1.45mm_HandSolder, F.Cu at (77.4, 150.7)
- added D2: SMBJ28CA, Diode_SMD:D_SMB, F.Cu at (32.4, 115.7)
- added D3: 1N4744A, Diode_THT:D_DO-41_SOD81_P7.62mm_Horizontal, F.Cu at (37.8, 118.9)
- added F1: PPTC 3A, Fuse:Fuse_Bourns_MF-RG300, F.Cu at (37.6, 112.7)
- added Q1: IRF4905, Package_TO_SOT_THT:TO-220-3_Vertical, F.Cu at (48.9, 114.9)
- added R38: 10k, Resistor_SMD:R_0805_2012Metric_Pad1.20x1.40mm_HandSolder, F.Cu at (62.4, 150.7)
- added R39: 10k, Resistor_SMD:R_0805_2012Metric_Pad1.20x1.40mm_HandSolder, F.Cu at (67.4, 150.7)
- added R40: 47k, Resistor_SMD:R_0805_2012Metric_Pad1.20x1.40mm_HandSolder, F.Cu at (72.4, 150.7)
- added R41: 10k, Resistor_SMD:R_0805_2012Metric_Pad1.20x1.40mm_HandSolder, F.Cu at (51.4, 119.2)
- added U3: 74HC123, Package_DIP:DIP-16_W7.62mm_Socket, F.Cu at (75.3, 120.2)
- added U4: 74HCT245, Package_DIP:DIP-20_W7.62mm_Socket, F.Cu at (35.4, 50.7)
- Q2, Q3, Q4, Q5, Q6, Q7, Q8, Q9: footprint ULN2803APG:DIP762W55P254L2286H480Q18N -> Package_DIP:DIP-18_W7.62mm_Socket
- U10, U11, U12, U13, U14, U25, U26, U27, U30, U31, U32, U5, U6, U7, U8, U9: footprint ULN2803APG:74HC595n -> Package_DIP:DIP-16_W7.62mm_Socket
- U15, U16, U17, U18, U19, U33, U34, U35: footprint UDN2981A:DIP254P762X533-18 -> Package_DIP:DIP-18_W7.62mm_Socket
- U22: footprint 74HC00N:DIP254P762X420-14 -> Package_DIP:DIP-14_W7.62mm_Socket
- moved U15 87.4 mm to (189.1, 72.7)
- moved U16 87.4 mm to (166.3, 72.7)
- moved U17 87.4 mm to (143.4, 72.7)
- moved U18 87.4 mm to (120.5, 72.7)
- moved U33 87.4 mm to (212.0, 72.7)
- moved U34 87.4 mm to (234.8, 72.7)
- moved U35 87.4 mm to (257.7, 72.7)
- moved U19 87.4 mm to (97.7, 72.7)
- moved U22 86.8 mm to (64.4, 120.2)
- moved Q7 80.8 mm to (200.5, 72.7)
- moved Q2 80.8 mm to (177.7, 72.7)
- moved Q3 80.8 mm to (154.8, 72.7)
- moved Q9 80.8 mm to (246.3, 72.7)
- moved Q5 80.8 mm to (109.1, 72.7)
- moved Q4 80.8 mm to (132.0, 72.7)
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Connections:
- C10 pad 1: +3.3V -> +5V
- C11 pad 1: +3.3V -> +5V
- C12 pad 1: +3.3V -> +5V
- C13 pad 2: +3.3V -> +5V
- C14 pad 1: +3.3V -> +5V
- C15 pad 1: +3.3V -> +5V
- C16 pad 2: +3.3V -> +5V
- C2 pad 1: +3.3V -> +5V
- C27 pad 2: +3.3V -> +5V
- C28 pad 2: +3.3V -> +5V
- C32 pad 2: +3.3V -> +5V
- C33 pad 2: +3.3V -> +5V
- C34 pad 2: +3.3V -> +5V
- C35 pad 1: +3.3V -> +5V
- C36 pad 1: +3.3V -> +5V
- C37 pad 1: +3.3V -> +5V
- C6 pad 1: +3.3V -> +5V
- C9 pad 1: +3.3V -> +5V
- J1 pad 1: +24V -> /VIN_RAW
- J11 pad 1: Net-(J11-Pin_1) -> /ESP_3V3
- J8 pad 1: +3.3V -> /ESP_3V3
- J9 pad 1: +24V -> /VIN_RAW
- U10 pad 10: /Clear -> /Clear_5V
- U10 pad 11: /Clock -> /Clock_5V
- U10 pad 12: /Column_Latch -> /Column_Latch_5V
- U10 pad 13: Net-(U10-~{OE}) -> /SR_N
- U10 pad 16: +3.3V -> +5V
- U11 pad 10: /Clear -> /Clear_5V
- U11 pad 11: /Clock -> /Clock_5V
- U11 pad 12: /Column_Latch -> /Column_Latch_5V
- U11 pad 13: Net-(U10-~{OE}) -> /SR_N
- U11 pad 16: +3.3V -> +5V
- U12 pad 10: /Clear -> /Clear_5V
- U12 pad 11: /Clock -> /Clock_5V
- U12 pad 12: /Column_Latch -> /Column_Latch_5V
- U12 pad 13: Net-(U10-~{OE}) -> /SR_N
- U12 pad 16: +3.3V -> +5V
- U13 pad 10: /Clear -> /Clear_5V
- U13 pad 11: /Clock -> /Clock_5V
- U13 pad 12: /Column_Latch -> /Column_Latch_5V
- U13 pad 13: Net-(U10-~{OE}) -> /SR_N
- U13 pad 16: +3.3V -> +5V
- U14 pad 10: /Clear -> /Clear_5V
- U14 pad 11: /Clock -> /Clock_5V
- U14 pad 12: /Column_Latch -> /Column_Latch_5V
- U14 pad 13: Net-(U10-~{OE}) -> /SR_N
- U14 pad 14: /Data -> /Data_5V
- U14 pad 16: +3.3V -> +5V
- U22 pad 1: Net-(U20-1Q) -> /Set_Reset_5V
- U22 pad 10: unconnected-(U22-Pad10) -> /Set_Reset_5V
- U22 pad 14: +3.3V -> +5V
- U22 pad 2: /Pulse -> /Pulse_Gated
- U22 pad 4: Net-(U10-~{OE}) -> /SR_N
- U22 pad 5: /Pulse -> /Pulse_Gated
- U22 pad 8: unconnected-(U22-Pad8) -> /SR_N
- U22 pad 9: unconnected-(U22-Pad9) -> /Set_Reset_5V
- U23 pad 1: Net-(J11-Pin_1) -> /ESP_3V3
- U25 pad 10: /Clear -> /Clear_5V
- U25 pad 11: /Clock -> /Clock_5V
- U25 pad 12: /Row_Latch -> /Row_Latch_5V
- U25 pad 16: +3.3V -> +5V
- U26 pad 10: /Clear -> /Clear_5V
- U26 pad 11: /Clock -> /Clock_5V
- U26 pad 12: /Row_Latch -> /Row_Latch_5V
- U26 pad 16: +3.3V -> +5V
- U27 pad 10: /Clear -> /Clear_5V
- U27 pad 11: /Clock -> /Clock_5V
- U27 pad 12: /Row_Latch -> /Row_Latch_5V
- U27 pad 14: /Data -> /Data_5V
- U27 pad 16: +3.3V -> +5V
- U30 pad 10: /Clear -> /Clear_5V
- U30 pad 11: /Clock -> /Clock_5V
- U30 pad 12: /Row_Latch -> /Row_Latch_5V
- U30 pad 16: +3.3V -> +5V
- U31 pad 10: /Clear -> /Clear_5V
- U31 pad 11: /Clock -> /Clock_5V
- U31 pad 12: /Row_Latch -> /Row_Latch_5V
- U31 pad 16: +3.3V -> +5V
- U32 pad 10: /Clear -> /Clear_5V
- U32 pad 11: /Clock -> /Clock_5V
- U32 pad 12: /Row_Latch -> /Row_Latch_5V
- U32 pad 14: /Data -> /Data_5V
- U32 pad 16: +3.3V -> +5V
- U5 pad 10: /Clear -> /Clear_5V
- U5 pad 11: /Clock -> /Clock_5V
- U5 pad 12: /Column_Latch -> /Column_Latch_5V
- U5 pad 16: +3.3V -> +5V
- U6 pad 10: /Clear -> /Clear_5V
- U6 pad 11: /Clock -> /Clock_5V
- U6 pad 12: /Column_Latch -> /Column_Latch_5V
- U6 pad 16: +3.3V -> +5V
- U7 pad 10: /Clear -> /Clear_5V
- U7 pad 11: /Clock -> /Clock_5V
- U7 pad 12: /Column_Latch -> /Column_Latch_5V
- U7 pad 16: +3.3V -> +5V
- U8 pad 10: /Clear -> /Clear_5V
- U8 pad 11: /Clock -> /Clock_5V
- U8 pad 12: /Column_Latch -> /Column_Latch_5V
- U8 pad 16: +3.3V -> +5V
- U9 pad 10: /Clear -> /Clear_5V
- U9 pad 11: /Clock -> /Clock_5V
- U9 pad 12: /Column_Latch -> /Column_Latch_5V
- U9 pad 14: /Data -> /Data_5V
- U9 pad 16: +3.3V -> +5V
Routing:
- net +5V: track 150.1 -> 687.0 mm, vias 1 -> 5
- net +3.3V: track 524.8 -> 0.00 mm, vias 3 -> 0
- net /Clock_5V: track 0.00 -> 345.9 mm, vias 0 -> 2
- net /Clear_5V: track 0.00 -> 312.8 mm
- net /Row_Latch_5V: track 0.00 -> 298.1 mm, vias 0 -> 3
- net /Data_5V: track 0.00 -> 289.5 mm, vias 0 -> 2
- net /Clear: track 301.4 -> 21.4 mm, vias 3 -> 0
- net /Row_Latch: track 285.9 -> 27.0 mm, vias 3 -> 0
- net /Column_Latch_5V: track 0.00 -> 237.0 mm, vias 0 -> 2
- net /Clock: track 298.6 -> 92.5 mm, vias 0 -> 1
- net /Column_Latch: track 223.3 -> 27.8 mm, vias 2 -> 0
- net GND1: track 1045.0 -> 1235.8 mm, vias 5 -> 10
- net Net-(U10-~{OE}): track 173.9 -> 0.00 mm, vias 3 -> 0
- net /SR_N: track 0.00 -> 129.7 mm
- net /Set_Reset_5V: track 0.00 -> 125.3 mm, vias 0 -> 1
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Other:
- board text added: "PULSE LIMIT"
- board text removed: "+3.3V"
- board text removed: "3.3V LDO"
