File: PCB_Controller/PCB_Controller.kicad_sch (KiCad schematic)
At the start: 141 parts, among them J1 ATX_Pin_fromPSU, J10 Conn_01x15, J11 Conn_01x15, J2 ColumnPin_1-12, J3 ColumnPin_13-24, J4 ColumnPin_25-36, J5 RowPin_1-8, J6 RowPin_9-16, J7 RowPin17-24, J8 Conn_01x05, Q2 ULN2803APG_O,N,HZN, Q3 ULN2803APG_O,N,HZN, Q4 ULN2803APG_O,N,HZN, Q5 ULN2803APG_O,N,HZN, Q6 ULN2803APG_O,N,HZN, Q7 ULN2803APG_O,N,HZN, Q8 ULN2803APG_O,N,HZN, Q9 ULN2803APG_O,N,HZN, U10 74HC595, U11 74HC595, U12 74HC595, U13 74HC595, U14 74HC595, U15 UDN2981A, U16 UDN2981A, U17 UDN2981A, U18 UDN2981A, U19 UDN2981A, U20 SN74HC75N, U22 74HC00, U23 ESP32-DEVKIT-V1, U25 74HC595, U26 74HC595, U27 74HC595, U30 74HC595, U31 74HC595, U32 74HC595, U33 UDN2981A, U34 UDN2981A, U35 UDN2981A, U5 74HC595, U6 74HC595, U7 74HC595, U8 74HC595, U9 74HC595

Commit message: Power the controller from a 24 V jack and shrink the board to 249x122 mm
- The ATX 20-pin input is gone. A 24 V barrel jack (CUI PJ-063AH, 8 A)
  feeds the coil drivers directly, with a 470 uF bulk cap. A TRACO
  TSR 1-2450 makes 5 V for the ESP32's VIN; the DevKit's 3V3 pin feeds
  the +3.3V logic rail. VIN used to sit on 3.3 V, which starved the
  DevKit's own regulator.
- One ground: GND2 was the ATX -12 V rail, which left the ULN2803
  emitters 12 V below the 74HC595 outputs driving them.
- The coil rail is +24V (was +12V). The PSU-status LED now shows 5 V,
  through 2.2k.
- PULSE moves to GPIO32 and SET/RST to GPIO33: GPIO34/35 are input-only
  and could not drive U22/U20.
- New layout, 249x122 mm (was 304x203): 16 channel strips of driver,
  pull-downs and 74HC595, the six IDC headers along the top edge, the
  ESP32 and power entry on the left. Autorouted with Freerouting, GND
  poured on both layers. Net classes: +24V 1.0 mm, GND 0.8 mm, coil
  lines 0.6 mm, logic power 0.5 mm, signals 0.3 mm, 0.3 mm clearance.
- DRC: no errors, nothing unconnected, matches the schematic.

Co-Authored-By: Claude Opus 5.5 <noreply@anthropic.com>
Parts:
- removed J1: ATX_Pin_fromPSU, ATX:39-29-920Y, symbol 39-29-9202:39-29-9202
- added C1: 470uF/35V, Capacitor_THT:CP_Radial_D10.0mm_P5.00mm, symbol Device:C_Polarized_Small
- added C3: 10uF/50V, Capacitor_SMD:C_1206_3216Metric_Pad1.33x1.80mm_HandSolder, symbol Device:C_Small
- added C4: 22uF/10V, Capacitor_SMD:C_1206_3216Metric_Pad1.33x1.80mm_HandSolder, symbol Device:C_Small
- added J1: 24V_DC_Jack, Connector_BarrelJack:BarrelJack_CUI_PJ-063AH_Horizontal, symbol Connector:Barrel_Jack
- added U1: TSR_1-2450, Converter_DCDC:Converter_DCDC_TRACO_TSR-1_THT, symbol Converter_DCDC:TSR_1-2450
- D1: value LED_PSU_Status -> LED_Power_5V
- R1: value 10k -> 2.2k
Connections:
- net Checker is gone; now on net +5V: R1.1
- net D32 is gone; now on net Pulse: J10.10 (Pin_10), U23.21 (D32)
- net D33 is gone; now on net Set_Reset: J10.9 (Pin_9), U23.22 (D33)
- net GND2 is gone; now on net GND1: C17.1, C18.1, C19.1, C20.1, C21.2, C22.1, C23.1, C24.1, C25.1, C26.2, C29.2, C30.2, C31.2, C38.2, C39.2, C40.1, J8.5 (Pin_5), Q2.9 (GND), Q3.9 (GND), Q4.9 (GND), Q5.9 (GND), Q6.9 (GND), Q7.9 (GND), Q8.9 (GND), Q9.9 (GND), U15.10 (GND), U16.10 (GND), U17.10 (GND), U18.10 (GND), U19.10 (GND), U33.10 (GND), U34.10 (GND), U35.10 (GND)
- net +3.3V: now also J11.1 (Pin_1), U23.1 (3V3); no longer U23.30 (VIN)
- net +5V: now also U23.30 (VIN), C4.1, U1.3 (Vout)
- net GND1: now also C1.2, C3.2, C4.2, J1.2, U1.2 (GND)
- net Pulse: no longer J10.12 (Pin_12), U23.19 (D34)
- net Set_Reset: no longer J10.11 (Pin_11), U23.20 (D35)
- net +12V renamed +24V
- net +24V: now also C1.1, C3.1, J1.1, U1.1 (Vin)
- new net D34: J10.12 (Pin_12), U23.19 (D34)
- new net D35: J10.11 (Pin_11), U23.20 (D35)
- no-connect marks 57 -> 55

Commit message: Add a 3.3 V LDO and a 24 V screw terminal to the controller power input
- J1 is now a 5.5 x 2.5 mm jack (CUI PJ-063BH, 8 A) to match 24 V
  10 A / 20 A adapter plugs; same land pattern as before
- J9: 2-pole 5.08 mm screw terminal in parallel with J1 for supplies
  with bare leads
- U2 AMS1117-3.3 (C5/C7) makes the +3.3V logic rail from +5V for the
  74HC595s, 74HC00 and 74HC75, instead of borrowing the DevKit's LDO
- The DevKit 3V3 pin is off the board rail (broken out on J11.1 only)
- J10.1, which sits on the ESP32 VIN pin, is now on +5V like VIN
- Re-placed and re-routed with Freerouting: DRC 0 errors, 0 unconnected

Co-Authored-By: Claude Opus 5.5 <noreply@anthropic.com>
Parts:
- added C5: 10uF/16V, Capacitor_SMD:C_1206_3216Metric_Pad1.33x1.80mm_HandSolder, symbol Device:C_Small
- added C7: 22uF/10V, Capacitor_SMD:C_1206_3216Metric_Pad1.33x1.80mm_HandSolder, symbol Device:C_Small
- added J9: Screw_Terminal_24V, TerminalBlock_Phoenix:TerminalBlock_Phoenix_MKDS-1,5-2-5.08_1x02_P5.08mm_Horizontal, symbol Connector:Screw_Terminal_01x02
- added U2: AMS1117-3.3, Package_TO_SOT_SMD:SOT-223-3_TabPin2, symbol Regulator_Linear:AMS1117-3.3
- J1: value 24V_DC_Jack -> DC_Jack_5.5x2.5_24V
Connections:
- net +24V: now also J9.1 (Pin_1)
- net +3.3V: now also C7.1, U2.2 (VO); no longer J10.1 (Pin_1), J11.1 (Pin_1), U23.1 (3V3)
- net +5V: now also J10.1 (Pin_1), C5.1, U2.3 (VI)
- net GND1: now also C5.2, C7.2, J9.2 (Pin_2), U2.1 (GND)
- new net: J11.1 (Pin_1), U23.1 (3V3)
Other:
- moved on the sheet: C4

Commit message: Buffer the ESP32, cap coil pulses in hardware and protect the 24 V input
- U4 74HCT245 turns the ESP32's 3.3 V control lines into 5 V for all
  logic, so the 595s, 74HC00 and 74HC123 can be HC or HCT parts
- All logic now runs on +5V (74HC595 at 3.3 V could not drive a ULN2803
  channel to the ~0.5 A a coil pulse needs); AMS1117 and the 3.3 V rail
  are gone, J8 pin 1 / J11 pin 1 break out the DevKit's own 3V3
- U3 74HC123 one-shot: drivers see PULSE for at most ~2 ms (R40/C8)
- 10k pull-downs on PULSE and SET/RST keep the drivers off at boot
- 74HC75 (latch tied transparent) replaced by a spare 74HC00 gate
- Input: PPTC 3 A (F1), SMBJ28CA TVS (D2), IRF4905 reverse-polarity
  switch (Q1, D3 15 V zener, R41), 1000 uF bulk (C42)
- All 35 ICs on standard DIP socket footprints (the old 595 footprint
  had 7.94 mm rows), socket pads 1.4 mm to leave routing room
- Keepouts around the mounting holes; re-placed and re-routed, board
  kept at the position it was moved to in KiCad
- DRC 0 errors / 0 unconnected / 0 parity, ERC 0 errors
- ref/: the single-dot current pulse the limiter is sized for

Co-Authored-By: Claude Opus 5.5 <noreply@anthropic.com>
Parts:
- removed C5: 10uF/16V, Capacitor_SMD:C_1206_3216Metric_Pad1.33x1.80mm_HandSolder, symbol Device:C_Small
- removed C7: 22uF/10V, Capacitor_SMD:C_1206_3216Metric_Pad1.33x1.80mm_HandSolder, symbol Device:C_Small
- removed U2: AMS1117-3.3, Package_TO_SOT_SMD:SOT-223-3_TabPin2, symbol Regulator_Linear:AMS1117-3.3
- removed U20: SN74HC75N, SN74HC75N:7475, symbol SN74HC74N:SN74HC75N
- added C41, C43, C8: 100nF, Capacitor_SMD:C_0805_2012Metric_Pad1.18x1.45mm_HandSolder, symbol Device:C_Small
- added C42: 1000uF/35V, Capacitor_THT:CP_Radial_D12.5mm_P5.00mm, symbol Device:C_Polarized_Small
- added D2: SMBJ28CA, Diode_SMD:D_SMB, symbol Device:D_TVS
- added D3: 1N4744A, Diode_THT:D_DO-41_SOD81_P7.62mm_Horizontal, symbol Device:D_Zener
- added F1: PPTC 3A, Fuse:Fuse_Bourns_MF-RG300, symbol Device:Polyfuse
- added Q1: IRF4905, Package_TO_SOT_THT:TO-220-3_Vertical, symbol Transistor_FET:IRF4905
- added R38, R39, R41: 10k, Resistor_SMD:R_0805_2012Metric_Pad1.20x1.40mm_HandSolder, symbol Device:R_Small
- added R40: 47k, Resistor_SMD:R_0805_2012Metric_Pad1.20x1.40mm_HandSolder, symbol Device:R_Small
- added U3: 74HC123, Package_DIP:DIP-16_W7.62mm_Socket, symbol 74xx:74HC123
- added U4: 74HCT245, Package_DIP:DIP-20_W7.62mm_Socket, symbol 74xx:74HC245
- Q2, Q3, Q4, Q5, Q6, Q7, Q8, Q9: footprint ULN2803APG:DIP762W55P254L2286H480Q18N -> Package_DIP:DIP-18_W7.62mm_Socket
- U10, U11, U12, U13, U14, U25, U26, U27, U30, U31, U32, U5, U6, U7, U8, U9: footprint ULN2803APG:74HC595n -> Package_DIP:DIP-16_W7.62mm_Socket
- U15, U16, U17, U18, U19, U33, U34, U35: footprint UDN2981A:DIP254P762X533-18 -> Package_DIP:DIP-18_W7.62mm_Socket
- U22: footprint 74HC00N:DIP254P762X420-14 -> Package_DIP:DIP-14_W7.62mm_Socket
Connections:
- net +24V: now also C42.1, D3.1 (K), Q1.3 (S); no longer J1.1, J9.1 (Pin_1)
- net +5V: now also C10.1, C11.1, C12.1, C13.2, C14.1, C15.1, C16.2, C2.1, C27.2, C28.2, C32.2, C33.2, C34.2, C35.1, C36.1, C37.1, C6.1, C9.1, U10.16 (VCC), U11.16 (VCC), U12.16 (VCC), U13.16 (VCC), U14.16 (VCC), U22.14 (VCC), U25.16 (VCC), U26.16 (VCC), U27.16 (VCC), U30.16 (VCC), U31.16 (VCC), U32.16 (VCC), U5.16 (VCC), U6.16 (VCC), U7.16 (VCC), U8.16 (VCC), U9.16 (VCC), C41.1, C43.1, R40.1, U3.16 (VCC), U4.1 (A->B), U4.20 (VCC)
- net Clear: now also U4.6 (A4); no longer U10.10 (~{SRCLR}), U11.10 (~{SRCLR}), U12.10 (~{SRCLR}), U13.10 (~{SRCLR}), U14.10 (~{SRCLR}), U25.10 (~{SRCLR}), U26.10 (~{SRCLR}), U27.10 (~{SRCLR}), U30.10 (~{SRCLR}), U31.10 (~{SRCLR}), U32.10 (~{SRCLR}), U5.10 (~{SRCLR}), U6.10 (~{SRCLR}), U7.10 (~{SRCLR}), U8.10 (~{SRCLR}), U9.10 (~{SRCLR})
- net Clock: now also U4.3 (A1); no longer U10.11 (SRCLK), U11.11 (SRCLK), U12.11 (SRCLK), U13.11 (SRCLK), U14.11 (SRCLK), U25.11 (SRCLK), U26.11 (SRCLK), U27.11 (SRCLK), U30.11 (SRCLK), U31.11 (SRCLK), U32.11 (SRCLK), U5.11 (SRCLK), U6.11 (SRCLK), U7.11 (SRCLK), U8.11 (SRCLK), U9.11 (SRCLK)
- net Column_Latch: now also U4.4 (A2); no longer U10.12 (RCLK), U11.12 (RCLK), U12.12 (RCLK), U13.12 (RCLK), U14.12 (RCLK), U5.12 (RCLK), U6.12 (RCLK), U7.12 (RCLK), U8.12 (RCLK), U9.12 (RCLK)
- net Data: now also U4.2 (A0); no longer U14.14 (SER), U27.14 (SER), U32.14 (SER), U9.14 (SER)
- net GND1: now also C41.2, C42.2, C43.2, D2.2 (A2), R38.2, R39.2, R41.2, U3.1 (A), U3.10 (B), U3.11 (Clr), U3.8 (GND), U3.9 (A), U4.10 (GND), U4.19 (CE), U4.9 (A7)
- net Pulse: now also R38.1, U4.7 (A5); no longer U22.2, U22.5
- net Row_Latch: now also U4.5 (A3); no longer U25.12 (RCLK), U26.12 (RCLK), U27.12 (RCLK), U30.12 (RCLK), U31.12 (RCLK), U32.12 (RCLK)
- net Set_Reset: now also R39.1, U4.8 (A6)
- net SR_N: now reaches U10.13 (~{OE}), U11.13 (~{OE}), U12.13 (~{OE}), U13.13 (~{OE}), U14.13 (~{OE}), U22.4
- net SR_N: now also U22.8
- net ESP_3V3: now reaches J11.1 (Pin_1), U23.1 (3V3)
- net ESP_3V3: now also J8.1 (Pin_1)
- net Set_Reset_5V: now reaches U22.1
- net Set_Reset_5V: now also U22.10, U22.9, U4.12 (B6)
- removed net +3.3V: C10.1, C11.1, C12.1, C13.2, C14.1, C15.1, C16.2, C2.1, C27.2, C28.2, C32.2, C33.2, C34.2, C35.1, C36.1, C37.1, C6.1, C9.1, J8.1 (Pin_1), U10.16 (VCC), U11.16 (VCC), U12.16 (VCC), U13.16 (VCC), U14.16 (VCC), U22.14 (VCC), U25.16 (VCC), U26.16 (VCC), U27.16 (VCC), U30.16 (VCC), U31.16 (VCC), U32.16 (VCC), U5.16 (VCC), U6.16 (VCC), U7.16 (VCC), U8.16 (VCC), U9.16 (VCC)
- new net Clear_5V: U10.10 (~{SRCLR}), U11.10 (~{SRCLR}), U12.10 (~{SRCLR}), U13.10 (~{SRCLR}), U14.10 (~{SRCLR}), U25.10 (~{SRCLR}), U26.10 (~{SRCLR}), U27.10 (~{SRCLR}), U30.10 (~{SRCLR}), U31.10 (~{SRCLR}), U32.10 (~{SRCLR}), U4.14 (B4), U5.10 (~{SRCLR}), U6.10 (~{SRCLR}), U7.10 (~{SRCLR}), U8.10 (~{SRCLR}), U9.10 (~{SRCLR})
- new net Clock_5V: U10.11 (SRCLK), U11.11 (SRCLK), U12.11 (SRCLK), U13.11 (SRCLK), U14.11 (SRCLK), U25.11 (SRCLK), U26.11 (SRCLK), U27.11 (SRCLK), U30.11 (SRCLK), U31.11 (SRCLK), U32.11 (SRCLK), U4.17 (B1), U5.11 (SRCLK), U6.11 (SRCLK), U7.11 (SRCLK), U8.11 (SRCLK), U9.11 (SRCLK)
- new net Column_Latch_5V: U10.12 (RCLK), U11.12 (RCLK), U12.12 (RCLK), U13.12 (RCLK), U14.12 (RCLK), U4.16 (B2), U5.12 (RCLK), U6.12 (RCLK), U7.12 (RCLK), U8.12 (RCLK), U9.12 (RCLK)
- new net Data_5V: U14.14 (SER), U27.14 (SER), U32.14 (SER), U4.18 (B0), U9.14 (SER)
- new net MONO_C: C8.2, U3.14 (Cext)
- new net MONO_RC: C8.1, R40.2, U3.15 (RCext)
- new net Pulse_5V: U3.2 (B), U3.3 (Clr), U4.13 (B5)
- new net Pulse_Gated: U22.2, U22.5, U3.13 (Q)
- new net Q1_GATE: D3.2 (A), Q1.1 (G), R41.1
- new net Row_Latch_5V: U25.12 (RCLK), U26.12 (RCLK), U27.12 (RCLK), U30.12 (RCLK), U31.12 (RCLK), U32.12 (RCLK), U4.15 (B3)
- new net VIN_FUSED: D2.1 (A1), F1.2, Q1.2 (D)
- new net VIN_RAW: F1.1, J1.1, J9.1 (Pin_1)
- no-connect marks 55 -> 49
Other:
- note removed: "Reset"
- note removed: "Set"
